Commit message: improved odom

File: description/lidar.xacro (robot description, xacro)
@@ -4,5 +4,5 @@
         <parent link="chassis"/>
         <child link="laser_frame"/>
-        <origin xyz="0.35 0 0.23" rpy="3.14159 0 0"/>
+        <origin xyz="0.37 0 0.23" rpy="3.14159 0 0"/>
     </joint>
     <link name="laser_frame">

Commit message: adjusted lidar location to be more accurate

File: description/lidar.xacro (robot description, xacro)
@@ -4,5 +4,5 @@
         <parent link="chassis"/>
         <child link="laser_frame"/>
-        <origin xyz="0.37 0 0.23" rpy="3.14159 0 0"/>
+        <origin xyz="0.385 0 0.23" rpy="3.14159 0 0"/>
     </joint>
     <link name="laser_frame">

Commit message: adjusted speeds

File: description/lidar.xacro (robot description, xacro)
@@ -4,5 +4,5 @@
         <parent link="chassis"/>
         <child link="laser_frame"/>
-        <origin xyz="0.385 0 0.23" rpy="3.14159 0 0"/>
+        <origin xyz="0.45 0 0.23" rpy="3.14159 0 0"/>
     </joint>
     <link name="laser_frame">
