Commit message: not actually sure, just commiting to be safe

File: description/robot_core.xacro (robot description, xacro)
@@ -16,5 +16,5 @@
     <xacro:property name="caster_wheel_offset_x" value="0.375"/>
     <xacro:property name="caster_wheel_offset_z" value="${wheel_offset_z}"/>
-    <material name="white">
+    <material name="white">a
         <color rgba="1 1 1 1" />
     </material>

Commit message: adjusted wheel seperation

File: description/robot_core.xacro (robot description, xacro)
@@ -10,5 +10,5 @@
     <xacro:property name="wheel_mass" value="2.2"/>
     <xacro:property name="wheel_offset_x" value="0.04"/>
-    <xacro:property name="wheel_offset_y" value="0.2"/>
+    <xacro:property name="wheel_offset_y" value="0.225"/>
     <xacro:property name="wheel_offset_z" value="0.01"/>
     <xacro:property name="caster_wheel_radius" value="0.125"/>
@@ -16,5 +16,5 @@
     <xacro:property name="caster_wheel_offset_x" value="0.375"/>
     <xacro:property name="caster_wheel_offset_z" value="${wheel_offset_z}"/>
-    <material name="white">a
+    <material name="white">
         <color rgba="1 1 1 1" />
     </material>

File: description/ros2_control.xacro (robot description, xacro)
@@ -11,5 +11,5 @@
                 <param name="baud_rate">57600</param>
                 <param name="timeout_ms">1000</param>
-                <param name="enc_counts_per_rev">2786.2</param>
+                <param name="enc_counts_per_rev">5000</param>
             </hardware>
             <joint name="left_wheel_joint">
