Commit message: Changed Naming Conventions for better rtab support?

File: description/depth_camera.xacro (robot description, xacro)
@@ -16,8 +16,8 @@
     <joint name="camera_optical_joint" type="fixed">
         <parent link="camera_link"/>
-        <child link="camera_link_optical"/>
+        <child link="camera_color_optical_frame"/>
         <origin xyz="0 0 0" rpy="${-pi/2} 0 ${-pi/2}"/>
     </joint>
-    <link name="camera_link_optical"></link>
+    <link name="camera_color_optical_frame"></link>
     <gazebo reference="camera_link">
         <material>Gazebo/Red</material>
@@ -39,5 +39,5 @@
             </camera>
             <plugin name="camera_controller" filename="libgazebo_ros_camera.so">
-                <frame_name>camera_link_optical</frame_name>
+                <frame_name>camera_color_optical_frame</frame_name>
                 <min_depth>0.1</min_depth>
                 <max_depth>100.0</max_depth>

File: description/robot_core.xacro (robot description, xacro)
@@ -36,6 +36,6 @@
     <!-- BASE_FOOTPRINT LINK -->
     <joint name="base_footprint_joint" type="fixed">
-        <parent link="base_link"/>
-        <child link="base_footprint"/>
+        <parent link="base_footprint"/>
+        <child link="base_link"/>
         <origin xyz="0 0 0" rpy="0 0 0"/>
     </joint>
